File: PCB/starBi.kicad_pcb (KiCad board)
At the start: 2 copper layers, 109.7 x 80 mm, 10 parts, among them J1 Conn_01x04_Pin, J2 Conn_01x08_Pin, SW1 SW_Push, SW2 SW_Push, U1 XIAO-ESP32-C3-SMD, U2 DHT11

Commit message: Add files via upload
Parts:
- G*** (x2): moved to B.Cu
- moved G*** 40.3 mm to (169.4, 84.2)
- moved G*** 10.8 mm to (195.0, 97.1), turned to 180 degrees
- turned G*** to 180 degrees
